File: devboard.kicad_pcb (KiCad board)
At the start: 4 copper layers, 23.8 x 44.3 mm, 41 parts, among them J1 USB-C, J2 microSD, J4 GPIO-A, J5 GPIO-B, J6 GPIO-C, J7 DBG-PWR, SW1 RESET, SW2 BOOT0, SW3 USER, U1 STM32F411CEU6, U2 AP2112K-3.3, Y1 25MHz

Commit message: devlog 05
Parts:
- C2: value GND -> 18p
Other:
- board text added: "Designed by EVV"
- board text added: "Half Life - Hack Club"
Changed lines of the file:
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@@
 			)
 		)
-		(property "Value" "GND"
+		(property "Value" "18p"
 			(at 0 -1.16 0)
 			(layer "B.Fab")
@@
 		(layer "Edge.Cuts")
 	)
+	(gr_text "Half Life - Hack Club"
+		(at 155.8 111.6 0)
+		(layer "B.SilkS")
+		(effects
+			(font
+				(size 0.7 0.7)
+				(thickness 0.1)
+			)
+			(justify left bottom mirror)
+		)
+	)
+	(gr_text "Designed by EVV"
+		(at 156.1 110.35 0)
+		(layer "B.SilkS")
+		(effects
+			(font
+				(size 1 1)
+				(thickness 0.2)
+			)
+			(justify left bottom mirror)
+		)
+	)
 	(segment
